Commit message: modify the conversion from angle to radian in xacro

File: velodyne_description/urdf/Lidar.urdf.xacro (robot description, xacro)
@@ -1,6 +1,5 @@
 <?xml version="1.0"?>
 <robot xmlns:xacro="http://www.ros.org/wiki/xacro" name="LIDAR">
-  <xacro:property name="M_PI" value="3.1415926535897931" />
-  <xacro:macro name="Lidar" params="*origin parent:=base_link name:=lidar topic:=/scan organize_cloud:=false hz:=10 lasers:=16 samples:=1875 collision_range:=0.3 min_range:=0.9 max_range:=130.0 noise:=0.008 min_horizonal_angle:=-${M_PI} max_horizonal_angle:=${M_PI} min_vertical_angle:=-${15.0*M_PI/180.0} max_vertical_angle:=${15.0*M_PI/180.0} gpu:=false">
+  <xacro:macro name="Lidar" params="*origin parent:=base_link name:=lidar topic:=/scan organize_cloud:=false hz:=10 lasers:=16 samples:=1875 collision_range:=0.3 min_range:=0.9 max_range:=130.0 noise:=0.008 min_horizonal_angle:=${radians(-180)} max_horizonal_angle:=${radians(180)} min_vertical_angle:=${radians(-15.0)} max_vertical_angle:=${radians(15.0)} gpu:=false">
     <joint name="${name}_base_mount_joint" type="fixed">
       <xacro:insert_block name="origin" />

File: velodyne_description/urdf/example.urdf.xacro (robot description, xacro)
@@ -42,6 +42,6 @@
   <!-- <xacro:include filename="$(find velodyne_description)/urdf/Lidar.urdf.xacro"/>
   <xacro:Lidar parent="base_link" name="lidar" topic="/scan" hz="10" organize_cloud="${organize_cloud}" gpu="${gpu}"
-  samples="480" min_horizonal_angle="-${60.0*M_PI/180.0}" max_horizonal_angle="${60.0*M_PI/180.0}"
-  lasers="96" min_vertical_angle="-${12.5*M_PI/180.0}" max_vertical_angle="${12.5*M_PI/180.0}">
+  samples="480" min_horizonal_angle="-${radians(60.0)}" max_horizonal_angle="${radians(60.0)}"
+  lasers="96" min_vertical_angle="-${radians(12.5)}" max_vertical_angle="${radians(12.5)}">
     <origin xyz="0 0 0.2" rpy="0 0 0" />
   </xacro:Lidar> -->

Commit message: modify the sequence of elements in velodyne msg

File: velodyne_description/urdf/Lidar.urdf.xacro (robot description, xacro)
@@ -1,5 +1,5 @@
 <?xml version="1.0"?>
 <robot xmlns:xacro="http://www.ros.org/wiki/xacro" name="LIDAR">
-  <xacro:macro name="Lidar" params="*origin parent:=base_link name:=lidar topic:=/scan organize_cloud:=false hz:=10 lasers:=16 samples:=1875 collision_range:=0.3 min_range:=0.9 max_range:=130.0 noise:=0.008 min_horizonal_angle:=${radians(-180)} max_horizonal_angle:=${radians(180)} min_vertical_angle:=${radians(-15.0)} max_vertical_angle:=${radians(15.0)} gpu:=false">
+  <xacro:macro name="Lidar" params="*origin parent:=base_link name:=lidar topic:=/scan organize_cloud:=false hz:=10 lasers:=16 samples:=1875 collision_range:=0.3 min_range:=0.9 max_range:=150.0 noise:=0.008 min_horizonal_angle:=${radians(-180)} max_horizonal_angle:=${radians(180)} min_vertical_angle:=${radians(-15.0)} max_vertical_angle:=${radians(15.0)} gpu:=false">
     <joint name="${name}_base_mount_joint" type="fixed">
       <xacro:insert_block name="origin" />
